File: pcb/ThermalCam.kicad_pcb (KiCad board)
At the start: 2 copper layers, 127 x 37 mm, 39 parts, among them J1 USB_B_Mini, SW2 SW_Push, SW3 SW_Push, U1 AMS1117-3.3, U2 AMG8833, U4 ESP32-WROOM-32, U5 ILI9341-HLG-18, U6 Arducam_SPI, U7 ESP32_PROG

Commit message: added eastrising 1.44 tft
Parts:
- BOOT1, SW2, SW3: footprint Button_Switch_SMD:SW_SPST_EVQP2 -> Button_Switch_SMD:SW_SPST_TL3342
- moved R11 1.95 mm to (152.0, 48.0)
- moved R12 1.95 mm to (152.0, 27.0)
- turned SW2 to 180 degrees
- turned SW3 to 0 degrees
- renumbered Re to R7
Routing:
- net GND: track 22.7 -> 34.8 mm, vias 16 -> 46
- net +3V3: track 287.3 -> 294.4 mm, vias 4 -> 6
- net BOOT0: track 59.4 -> 62.5 mm
- net Net-(R11-Pad1): track 8.69 -> 11.3 mm
- net Net-(R1-Pad2): track 11.3 -> 12.9 mm
- net BUTTON1: track 63.1 -> 64.1 mm
- net BUTTON0: track 48.5 -> 49.2 mm
- net +5V: track 4.46 -> 3.83 mm
- net Net-(BOOT1-Pad1): track 8.75 -> 9.36 mm

Commit message: update
Parts:
- removed U5: ILI9341-HLG-18, Connector_PinHeader_2.54mm:PinHeader_1x08_P2.54mm_Vertical
- added C1: 10uf, Capacitor_SMD:C_1206_3216Metric, F.Cu at (193.5, 42.0)
- added C12: 0.1uf, Capacitor_SMD:C_1206_3216Metric, F.Cu at (193.5, 32.5)
- added R13: 1K, Resistor_SMD:R_1206_3216Metric, F.Cu at (193.5, 37.5)
- added U3: ST7735S, EastRising:ER-CON26HT-1, F.Cu at (199.0, 37.8)
- C11: value 10uf -> 100nf
- C2: value 100uf -> 100nf
Connections:
- U4 pad 16: MOSI_TFT -> DATA_TFT
Routing:
- net MOSI_TFT: track 107.7 -> 0.00 mm
- net DATA_TFT: track 0.00 -> 98.9 mm, vias 0 -> 1
- net GND: track 34.8 -> 57.5 mm, vias 46 -> 43
- net CS_TFT: track 88.5 -> 98.0 mm, vias 1 -> 2
- net Net-(R13-Pad1): track 0.00 -> 9.24 mm
- net +3V3: track 294.4 -> 298.4 mm, vias 6 -> 8
- net RESET_TFT: track 77.6 -> 80.4 mm, vias 1 -> 3
- net SCLK_TFT: track 123.5 -> 122.2 mm, vias 1 -> 3
- net DC_TFT: track 85.1 -> 86.2 mm
- net (no net): vias 0 -> 1
Other:
- net class Default: clearance 0.4 -> 0.2; trace_width 0.4 -> 0.2; via_dia 0.6 -> 0.5
- net class Power added: clearance 0.2, trace_width 0.3, via_dia 0.6, via_drill 0.3
- rule trace_clearance: 0.4 -> 0.2
- board text removed: "DC"
- board text removed: "DISPLAY"
- board text removed: "RESET"
